File: PCB/RP-KEY.kicad_pcb (KiCad board)
At the start: 2 copper layers, 39.4 x 12 mm, 24 parts, among them J1 USB_A_PCB_Edge_receptacle, SW10 SW_Push, SW11 SW_Push, SW12 SW_Push, SW13 SW_Push, SW14 SW_Push, U1 RP2350A, U3 MCP1700x-330xxTT, Y2 ABM8-272-T3

Commit message: Add files via upload
Parts:
- added R4: 10k, Resistor_SMD:R_0402_1005Metric, F.Cu at (146.3, 113.2)
- added R5: 27ohm, Resistor_SMD:R_0402_1005Metric, F.Cu at (158.6, 111.8)
- added R6: 27ohm, Resistor_SMD:R_0402_1005Metric, F.Cu at (159.6, 111.8)
- added SW15: SW_Push, Button_Switch_SMD:SW_Tactile_SPST_NO_Straight_CK_PTS636Sx25SMTRLFS, F.Cu at (144.4, 117.1)
- moved C2 0.21 mm to (161.2, 110.8)
- moved C4 0.11 mm to (157.1, 111.0)
- moved L1 0.10 mm to (161.2, 112.0)
- moved C5 0.10 mm to (157.1, 112.0)
- moved R1 0.09 mm to (155.6, 111.7)
Connections:
- U1 pad 26: unconnected-(U1-RUN-Pad26) -> Net-(U1-RUN)
- U1 pad 51: D- -> Net-(U1-USB_DM)
- U1 pad 52: D+ -> Net-(U1-USB_DP)
Routing:
- net Net-(U1-RUN): track 0.00 -> 29.1 mm, vias 0 -> 4
- net GND: track 38.4 -> 52.8 mm, vias 4 -> 7
- net 3.3V: track 51.8 -> 54.9 mm, vias 5 -> 7
- net D-: track 28.7 -> 30.6 mm
- net D+: track 27.9 -> 29.8 mm
- net Net-(U1-USB_DP): track 0.00 -> 1.28 mm
- net Net-(U1-USB_DM): track 0.00 -> 1.26 mm
- net 5V: track 22.7 -> 23.4 mm

Commit message: Add files via upload
Parts:
- added C10: 10 uf, Capacitor_SMD:C_0402_1005Metric, F.Cu at (157.1, 112.3)
- added C11: 10 uf, Capacitor_SMD:C_0402_1005Metric, F.Cu at (153.1, 117.0)
- added C6: 10 uf, Capacitor_SMD:C_0402_1005Metric, F.Cu at (153.8, 120.6)
- added C7: 10 uf, Capacitor_SMD:C_0402_1005Metric, F.Cu at (164.0, 120.8)
- added C8: 10 uf, Capacitor_SMD:C_0402_1005Metric, F.Cu at (163.1, 117.0)
- added C9: 10 uf, Capacitor_SMD:C_0402_1005Metric, F.Cu at (163.1, 114.6)
- moved R2 1.13 mm to (152.4, 120.7)
- moved C5 0.70 mm to (157.1, 111.3)
- moved C4 0.53 mm to (157.1, 110.4)
- moved L1 0.41 mm to (161.3, 111.6)
- moved SW10 0.23 mm to (165.8, 117.0)
- moved C2 0.22 mm to (161.2, 110.6)
- moved SW11 0.20 mm to (170.1, 117.0)
- moved C29 0.09 mm to (151.4, 120.7)
- moved Y2 0.08 mm to (148.8, 120.0)
Connections:
- U1 pad 23: Net-(U1-DVDD-Pad23) -> unconnected-(U1-DVDD-Pad23)_2
- U1 pad 39: Net-(U1-DVDD-Pad23) -> unconnected-(U1-DVDD-Pad23)
- U1 pad 47: unconnected-(U1-VREG_PGND-Pad47) -> GND
- U1 pad 6: Net-(U1-DVDD-Pad23) -> unconnected-(U1-DVDD-Pad23)_1
Routing:
- net Net-(U1-DVDD-Pad23): track 15.2 -> 0.00 mm
- net (no net): track 0.00 -> 15.2 mm
- net GND: track 52.8 -> 60.9 mm, vias 7 -> 10
- net 3.3V: track 54.9 -> 60.3 mm, vias 7 -> 8
- net /VREG_LX: track 5.59 -> 4.15 mm
- net Net-(C29-Pad1): track 4.04 -> 3.01 mm
- net XOUT: track 5.36 -> 6.33 mm
Other:
- outline, holes or cut-outs redrawn
