File: PCB/RP-KEY.kicad_sch (KiCad schematic)
At the start: 24 parts, among them J1 USB_A_PCB_Edge_receptacle, SW10 SW_Push, SW11 SW_Push, SW12 SW_Push, SW13 SW_Push, SW14 SW_Push, U1 RP2350A, U3 MCP1700x-330xxTT, Y2 ABM8-272-T3

Commit message: Add files via upload
Parts:
- added R4: 10k, Resistor_SMD:R_0402_1005Metric, symbol Device:R
- added R5, R6: 27ohm, Resistor_SMD:R_0402_1005Metric, symbol Device:R
- added SW15: SW_Push, Button_Switch_SMD:SW_Tactile_SPST_NO_Straight_CK_PTS636Sx25SMTRLFS, symbol Switch:SW_Push
Connections:
- net 3.3V: now also R4.2
- net D+: now also R5.2; no longer U1.52 (USB_DP)
- net D-: now also R6.2; no longer U1.51 (USB_DM)
- net GND: now also SW15.2
- net at U1.26 (RUN): now also R4.1, SW15.1
- new net: R6.1, U1.51 (USB_DM)
- new net: R5.1, U1.52 (USB_DP)
- no-connect marks 34 -> 33
Other:
- moved on the sheet: C29, C30, R2, Y2

Commit message: Add files via upload
Parts:
- added C10, C11, C6, C7, C8, C9: 10 uf, Capacitor_SMD:C_0402_1005Metric, symbol Device:C
Connections:
- net 3.3V: now also C10.1, C11.1, C6.1, C7.1, C8.1, C9.1
- net GND: now also U1.47 (VREG_PGND), C10.2, C11.2, C6.2, C7.2, C8.2, C9.2
- no-connect marks 33 -> 34
